File: Hardware/MP3/MP3.kicad_pcb (KiCad board)
At the start: 4 copper layers, 57 parts, among them IC1 MCP73871-2CCI_ML, IC2 AK4493SEQ, J1 Conn_02x20_Odd_Even, J2 USB_C_Receptacle_USB2.0, U1 TPS63000DRCR, U2 OPA1622IDRCR, Y1 ABM8-22.5792MHZ-D2Y-T

Commit message: feat: Changes to the power circuitry to sort out the regulators (schematic and footprint sorted). Additionally, headphone jack needs to be sorted, both schematic and actual component.
Parts:
- added C21: 1uF, Capacitor_SMD:C_0402_1005Metric, F.Cu at (156.5, 95.3)
- added C22: 1uF, Capacitor_SMD:C_0402_1005Metric, F.Cu at (161.8, 101.6)
- added C31: 1uF, Capacitor_SMD:C_0402_1005Metric, F.Cu at (151.6, 88.0)
- added C32: 1uF, Capacitor_SMD:C_0402_1005Metric, F.Cu at (157.0, 88.1)
- added C33: 1uF, Capacitor_SMD:C_0402_1005Metric, F.Cu at (151.2, 95.3)
- added C34: 1uF, Capacitor_SMD:C_0402_1005Metric, F.Cu at (156.5, 101.5)
- added C36: 10uF, Capacitor_SMD:C_0603_1608Metric, F.Cu at (127.7, 79.5)
- added J3: Conn_01x07_Pin, Connector_PinHeader_2.54mm:PinHeader_1x07_P2.54mm_Vertical, F.Cu at (139.8, 87.5)
- added U3: TPS7A20xxxDBV, Package_TO_SOT_SMD:SOT-23-5, F.Cu at (154.4, 88.6)
- added U4: TPS7A2033PDBVR, Package_TO_SOT_SMD:SOT-23-5, F.Cu at (153.9, 95.8)
- added U5: TPS7A20xxxDBV, Package_TO_SOT_SMD:SOT-23-5, F.Cu at (159.1, 102.1)
- moved U2 10.9 mm to (131.8, 80.1)
