File: Hardware/MP3/audio.kicad_sch (KiCad schematic)
At the start: 24 parts, among them IC2 AK4493SEQ, U2 OPA1622IDRCR, Y1 ABM8-22.5792MHZ-D2Y-T

Commit message: feat: Changes to the power circuitry to sort out the regulators (schematic and footprint sorted). Additionally, headphone jack needs to be sorted, both schematic and actual component.
Parts:
- added J5: AudioJack3_Ground_Switch, symbol Connector_Audio:AudioJack3_Ground_Switch
Connections:
- net GND: now also J5.G
Other:
- moved on the sheet: Y1
Changed lines of the file:
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@@
 	(text "Double check the pins, and add decoupling caps\nused for MCLK rather than DSP\n\nPins 1 and 3 are interchangable? so it seems\n\nCan't use this....\n"
 		(exclude_from_sim no)
-		(at 153.162 135.89 0)
+		(at 104.902 152.4 0)
 		(effects
 			(font
@@
 	)
 	(label "A3V3"
-		(at 166.37 154.94 0)
+		(at 118.11 171.45 0)
 		(effects
 			(font
@@
 	)
 	(label "AGND"
-		(at 135.89 154.94 180)
+		(at 87.63 171.45 180)
 		(effects
 			(font
@@
 	)
 	(label "AGND"
-		(at 166.37 157.48 0)
+		(at 118.11 173.99 0)
 		(effects
 			(font
@@
 	)
 	(label "CLOCK"
-		(at 147.32 127 180)
+		(at 99.06 143.51 180)
 		(effects
 			(font
@@
 	)
 	(label "CLOCK"
-		(at 135.89 157.48 180)
+		(at 87.63 173.99 180)
 		(effects
 			(font
@@
 	)
 	(symbol
+		(lib_id "Connector_Audio:AudioJack3_Ground_Switch")
+		(at 195.58 134.62 0)
+		(unit 1)
+		(exclude_from_sim no)
+		(in_bom yes)
+		(on_board yes)
+		(dnp no)
+		(fields_autoplaced yes)
+		(property "Reference" "J5"
+			(at 193.675 123.19 0)
+			(effects
+				(font
+					(size 1.27 1.27)
+				)
+			)
+		)
+		(property "Value" "AudioJack3_Ground_Switch"
+			(at 193.675 125.73 0)
+			(effects
+				(font
+					(size 1.27 1.27)
+				)
+			)
+		)
+		(property "Footprint" ""
+			(at 195.58 134.62 0)
+			(effects
+				(font
+					(size 1.27 1.27)
+				)
+				(hide yes)
+			)
+		)
+		(property "Datasheet" "~"
+			(at 195.58 134.62 0)
+			(effects
+				(font
+					(size 1.27 1.27)
+				)
+				(hide yes)
+			)
+		)
+		(property "Description" "Audio Jack, 3 Poles (Stereo / TRS), Grounded Sleeve, Switched Poles (Normalling)"
+			(at 195.58 134.62 0)
+			(effects
+				(font
+					(size 1.27 1.27)
+				)
+				(hide yes)
+			)
+		)
+		(pin "G"
+		)
+		(pin "TN"
+		)
+		(pin "S"
+		)
+		(pin "T"
+		)
+		(pin "R"
+		)
+		(pin "RN"
+		)
+		(pin "SN"
+		)
+		(instances
+			(project ""
+				(path "/0e2978a4-9114-4e8f-a3b0-a18c9ec8fe33/8299ee4d-961e-4056-9e41-08fab1b6f7ac"
+					(reference "J5")
+					(unit 1)
+				)
+			)
+		)
+	)
+	(symbol
 		(lib_id "power:+3.3V")
 		(at 35.56 21.59 0)
@@
 	(symbol
 		(lib_id "iclr:ABM8-22.5792MHZ-D2Y-T")
-		(at 166.37 157.48 180)
+		(at 118.11 173.99 180)
 		(unit 1)
 		(exclude_from_sim no)
@@
 		(fields_autoplaced yes)
 		(property "Reference" "Y1"
-			(at 151.13 147.32 0)
+			(at 102.87 163.83 0)
 			(effects
 				(font
@@
 		)
 		(property "Value" "ABM8-22.5792MHZ-D2Y-T"
-			(at 151.13 149.86 0)
+			(at 102.87 166.37 0)
 			(effects
 				(font
@@
 		)
 		(property "Footprint" "iclr:ABM810000MHZ12D2W"
-			(at 139.7 62.56 0)
+			(at 91.44 79.07 0)
 			(effects
 				(font
@@
 		)
 		(property "Datasheet" "https://abracon.com/Resonators/abm8.pdf"
-			(at 139.7 -37.44 0)
+			(at 91.44 -20.93 0)
 			(effects
 				(font
@@
 		)
 		(property "Description" "Crystal 22.5792MHz +/-20ppm (Tol) +/-30ppm (Stability) 18pF FUND 50Ohm 4-Pin Ultra Mini-CSMD T/R"
-			(at 166.37 157.48 0)
+			(at 118.11 173.99 0)
 			(effects
 				(font
@@
 		)
 		(property "Height" "0.8"
-			(at 139.7 -237.44 0)
+			(at 91.44 -220.93 0)
 			(effects
 				(font
@@
 		)
 		(property "Mouser Part Number" "N/A"
-			(at 139.7 -337.44 0)
+			(at 91.44 -320.93 0)
 			(effects
 				(font
@@
 		)
 		(property "Mouser Price/Stock" "https://www.mouser.com/Search/Refine.aspx?Keyword=N%2FA"
-			(at 139.7 -437.44 0)
+			(at 91.44 -420.93 0)
 			(effects
 				(font
@@
 		)
 		(property "Manufacturer_Name" "ABRACON"
-			(at 139.7 -537.44 0)
+			(at 91.44 -520.93 0)
 			(effects
 				(font
@@
 		)
 		(property "Manufacturer_Part_Number" "ABM8-22.5792MHZ-D2Y-T"
-			(at 139.7 -637.44 0)
+			(at 91.44 -620.93 0)
 			(effects
 				(font
@@
 					(unit 1)
 				)
+			)
+		)
+	)
+	(symbol
+		(lib_id "power:GND")
+		(at 195.58 147.32 0)
+		(unit 1)
+		(exclude_from_sim no)
+		(in_bom yes)
+		(on_board yes)
+		(dnp no)
+		(property "Reference" "#PWR056"
+			(at 195.58 153.67 0)
+			(effects
+				(font
+					(size 1.27 1.27)
+				)
+				(hide yes)
+			)
+		)
+		(property "Value" "GND"
+			(at 192.024 148.844 0)
+			(effects
+				(font
+					(size 1.27 1.27)
+				)
+			)
+		)
+		(property "Footprint" ""
+			(at 195.58 147.32 0)
+			(effects
+				(font
+					(size 1.27 1.27)
+				)
+				(hide yes)
+			)
+		)
+		(property "Datasheet" ""
+			(at 195.58 147.32 0)
+			(effects
+				(font
+					(size 1.27 1.27)
+				)
+				(hide yes)
+			)
+		)
+		(property "Description" ""
+			(at 195.58 147.32 0)
+			(effects
+				(font
+					(size 1.27 1.27)
+				)
+				(hide yes)
+			)
+		)
+		(pin "1"
+		)
+		(instances
+			(project "MP3"
+				(path "/0e2978a4-9114-4e8f-a3b0-a18c9ec8fe33/8299ee4d-961e-4056-9e41-08fab1b6f7ac"
+					(reference "#PWR056")
+					(unit 1)
+				)
